File: hardware/Scrutineering/Scrutineering.kicad_sch (KiCad schematic)
At the start: 22 parts, among them J1 Conn_02x04, J10 Conn_01x01, J11 Conn_01x02, J12 Conn_01x02, J2 Conn_02x04, J3 Conn_01x03, J4 Conn_01x03, J5 Conn_01x01, J6 Conn_01x01, J7 Conn_01x01, J8 Conn_01x01, J9 Conn_01x01

Commit message: changed to vertical connectors
Parts:
- J1, J2: footprint Scrutineering:nanofit_02x04 -> Scrutineering:CONN_SD-105310-100_08_MOL; P/N 1053141108 -> 1053101308
- J11, J12: footprint UTSVT_Connectors:105313-2102 -> UTSVT_Connectors:Molex_Nano-Fit_105309-xx02_1x02_P2.50mm_Vertical; P/N 1053131102 -> 1053091202
- J3, J4: footprint VoltTemp:1053131103 -> Scrutineering:CONN_SD-105309-100_03_MOL; P/N 1053131103 -> 1053091103
Changed lines of the file:
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@@
 			)
 		)
-		(property "Footprint" "UTSVT_Connectors:105313-2102"
+		(property "Footprint" "UTSVT_Connectors:Molex_Nano-Fit_105309-xx02_1x02_P2.50mm_Vertical"
 			(at 163.83 77.47 0)
 			(effects
@@
 			)
 		)
-		(property "P/N" "1053131102"
+		(property "P/N" "1053091202"
 			(at 163.83 77.47 0)
 			(effects
@@
 			)
 		)
-		(property "Footprint" "Scrutineering:nanofit_02x04"
+		(property "Footprint" "Scrutineering:CONN_SD-105310-100_08_MOL"
 			(at 71.12 87.63 0)
 			(effects
@@
 			)
 		)
-		(property "P/N" "1053141108"
+		(property "P/N" "1053101308"
 			(at 71.12 87.63 0)
 			(effects
@@
 			)
 		)
-		(property "Footprint" "Scrutineering:nanofit_02x04"
+		(property "Footprint" "Scrutineering:CONN_SD-105310-100_08_MOL"
 			(at 71.12 43.18 0)
 			(effects
@@
 			)
 		)
-		(property "P/N" "1053141108"
+		(property "P/N" "1053101308"
 			(at 71.12 43.18 0)
 			(effects
@@
 			)
 		)
-		(property "Footprint" "VoltTemp:1053131103"
+		(property "Footprint" "Scrutineering:CONN_SD-105309-100_03_MOL"
 			(at 109.22 87.63 0)
 			(effects
@@
 			)
 		)
-		(property "P/N" "1053131103"
+		(property "P/N" "1053091103"
 			(at 109.22 87.63 0)
 			(effects
@@
 			)
 		)
-		(property "Footprint" "VoltTemp:1053131103"
+		(property "Footprint" "Scrutineering:CONN_SD-105309-100_03_MOL"
 			(at 109.22 43.18 0)
 			(effects
@@
 			)
 		)
-		(property "P/N" "1053131103"
+		(property "P/N" "1053091103"
 			(at 109.22 43.18 0)
 			(effects
@@
 			)
 		)
-		(property "Footprint" "UTSVT_Connectors:105313-2102"
+		(property "Footprint" "UTSVT_Connectors:Molex_Nano-Fit_105309-xx02_1x02_P2.50mm_Vertical"
 			(at 185.42 69.85 0)
 			(effects
@@
 			)
 		)
-		(property "P/N" "1053131102"
+		(property "P/N" "1053091202"
 			(at 185.42 69.85 0)
 			(effects
