File: hardware/Scrutineering/Scrutineering.kicad_sch (KiCad schematic)
At the start: 22 parts, among them J1 Conn_02x04, J10 Conn_01x01, J11 Conn_01x02, J12 Conn_01x02, J2 Conn_02x04, J3 Conn_01x03, J4 Conn_01x03, J5 Conn_01x01, J6 Conn_01x01, J7 Conn_01x01, J8 Conn_01x01, J9 Conn_01x01

Commit message: Replaced Lakshay's tiny banana jacks with real ones
Parts:
- J10, J5, J6, J7, J8, J9: footprint UTSVT_Connectors:Banana_Jack_1_Pin_4mm -> VoltTemp:5754; P/N 105-2210-201 -> 575-4
Changed lines of the file:
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@@
 			)
 		)
-		(property "Footprint" "UTSVT_Connectors:Banana_Jack_1_Pin_4mm"
+		(property "Footprint" "VoltTemp:5754"
 			(at 72.39 69.85 0)
 			(effects
@@
 			)
 		)
-		(property "P/N" "105-2210-201"
+		(property "P/N" "575-4"
 			(at 72.39 69.85 0)
 			(effects
@@
 			)
 		)
-		(property "Footprint" "UTSVT_Connectors:Banana_Jack_1_Pin_4mm"
+		(property "Footprint" "VoltTemp:5754"
 			(at 140.97 86.36 0)
 			(effects
@@
 			)
 		)
-		(property "P/N" "105-2210-201"
+		(property "P/N" "575-4"
 			(at 140.97 86.36 90)
 			(effects
@@
 			)
 		)
-		(property "Footprint" "UTSVT_Connectors:Banana_Jack_1_Pin_4mm"
+		(property "Footprint" "VoltTemp:5754"
 			(at 53.34 97.79 0)
 			(effects
@@
 			)
 		)
-		(property "P/N" "105-2210-201"
+		(property "P/N" "575-4"
 			(at 53.34 97.79 90)
 			(effects
@@
 			)
 		)
-		(property "Footprint" "UTSVT_Connectors:Banana_Jack_1_Pin_4mm"
+		(property "Footprint" "VoltTemp:5754"
 			(at 54.61 52.07 0)
 			(effects
@@
 			)
 		)
-		(property "P/N" "105-2210-201"
+		(property "P/N" "575-4"
 			(at 54.61 52.07 90)
 			(effects
@@
 			)
 		)
-		(property "Footprint" "UTSVT_Connectors:Banana_Jack_1_Pin_4mm"
+		(property "Footprint" "VoltTemp:5754"
 			(at 140.97 71.12 0)
 			(effects
@@
 			)
 		)
-		(property "P/N" "105-2210-201"
+		(property "P/N" "575-4"
 			(at 140.97 71.12 90)
 			(effects
@@
 			)
 		)
-		(property "Footprint" "UTSVT_Connectors:Banana_Jack_1_Pin_4mm"
+		(property "Footprint" "VoltTemp:5754"
 			(at 72.39 116.84 0)
 			(effects
@@
 			)
 		)
-		(property "P/N" "105-2210-201"
+		(property "P/N" "575-4"
 			(at 72.39 116.84 0)
 			(effects
