File: hardware/Scrutineering/Scrutineering.kicad_sch (KiCad schematic)
At the start: 22 parts, among them J1 Conn_02x04, J10 Conn_01x01, J11 Conn_01x02, J12 Conn_01x02, J2 Conn_02x04, J3 Conn_01x03, J4 Conn_01x03, J5 Conn_01x01, J6 Conn_01x01, J7 Conn_01x01, J8 Conn_01x01, J9 Conn_01x01

Commit message: Scrutineering (#7)
* initial schematic and layout

* updated layout

* schematic with graphics/mounting

* graphics stuff

* fixed routing

* BOM and gerber (still need to find jack P/N)

* final

* revert back to main...

* added Scrutineering footprints

* added Scrutineering 3d models

* BOM and gerber with changed connector

* changed to vertical connectors

* added footprints/3d models vertical connectors

* fix 1 trace

* updated BOM

* updated BOM again

* Revert "fix 1 trace"

This reverts commit af0c854c5f9be3b18890f8714f235c97d2fe5d90.

:#

* Replaced Lakshay's tiny banana jacks with real ones

* fix unrouted

* Updated Gerbers

---------

Co-authored-by: Ravi Shah <ravidhruvishshah@gmail.com>
Co-authored-by: kretsdyl <kretschmandk@gmail.com>
Parts:
- J1, J2: footprint Scrutineering:nanofit_02x04 -> Scrutineering:CONN_SD-105310-100_08_MOL; P/N 1053141108 -> 1053101308
- J10, J5, J6, J7, J8, J9: footprint UTSVT_Connectors:Banana_Jack_1_Pin_4mm -> VoltTemp:5754; P/N 105-2210-201 -> 575-4
- J11, J12: footprint UTSVT_Connectors:105313-2102 -> UTSVT_Connectors:Molex_Nano-Fit_105309-xx02_1x02_P2.50mm_Vertical; P/N 1053131102 -> 1053091202
- J3, J4: footprint VoltTemp:1053131103 -> Scrutineering:CONN_SD-105309-100_03_MOL; P/N 1053131103 -> 1053091103
Changed lines of the file:
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@@
 			)
 		)
-		(property "Footprint" "UTSVT_Connectors:105313-2102"
+		(property "Footprint" "UTSVT_Connectors:Molex_Nano-Fit_105309-xx02_1x02_P2.50mm_Vertical"
 			(at 163.83 77.47 0)
 			(effects
@@
 			)
 		)
-		(property "P/N" "1053131102"
+		(property "P/N" "1053091202"
 			(at 163.83 77.47 0)
 			(effects
@@
 			)
 		)
-		(property "Footprint" "UTSVT_Connectors:Banana_Jack_1_Pin_4mm"
+		(property "Footprint" "VoltTemp:5754"
 			(at 72.39 69.85 0)
 			(effects
@@
 			)
 		)
-		(property "P/N" "105-2210-201"
+		(property "P/N" "575-4"
 			(at 72.39 69.85 0)
 			(effects
@@
 			)
 		)
-		(property "Footprint" "Scrutineering:nanofit_02x04"
+		(property "Footprint" "Scrutineering:CONN_SD-105310-100_08_MOL"
 			(at 71.12 87.63 0)
 			(effects
@@
 			)
 		)
-		(property "P/N" "1053141108"
+		(property "P/N" "1053101308"
 			(at 71.12 87.63 0)
 			(effects
@@
 			)
 		)
-		(property "Footprint" "Scrutineering:nanofit_02x04"
+		(property "Footprint" "Scrutineering:CONN_SD-105310-100_08_MOL"
 			(at 71.12 43.18 0)
 			(effects
@@
 			)
 		)
-		(property "P/N" "1053141108"
+		(property "P/N" "1053101308"
 			(at 71.12 43.18 0)
 			(effects
@@
 			)
 		)
-		(property "Footprint" "UTSVT_Connectors:Banana_Jack_1_Pin_4mm"
+		(property "Footprint" "VoltTemp:5754"
 			(at 140.97 86.36 0)
 			(effects
@@
 			)
 		)
-		(property "P/N" "105-2210-201"
+		(property "P/N" "575-4"
 			(at 140.97 86.36 90)
 			(effects
@@
 			)
 		)
-		(property "Footprint" "VoltTemp:1053131103"
+		(property "Footprint" "Scrutineering:CONN_SD-105309-100_03_MOL"
 			(at 109.22 87.63 0)
 			(effects
@@
 			)
 		)
-		(property "P/N" "1053131103"
+		(property "P/N" "1053091103"
 			(at 109.22 87.63 0)
 			(effects
@@
 			)
 		)
-		(property "Footprint" "VoltTemp:1053131103"
+		(property "Footprint" "Scrutineering:CONN_SD-105309-100_03_MOL"
 			(at 109.22 43.18 0)
 			(effects
@@
 			)
 		)
-		(property "P/N" "1053131103"
+		(property "P/N" "1053091103"
 			(at 109.22 43.18 0)
 			(effects
@@
 			)
 		)
-		(property "Footprint" "UTSVT_Connectors:Banana_Jack_1_Pin_4mm"
+		(property "Footprint" "VoltTemp:5754"
 			(at 53.34 97.79 0)
 			(effects
@@
 			)
 		)
-		(property "P/N" "105-2210-201"
+		(property "P/N" "575-4"
 			(at 53.34 97.79 90)
 			(effects
@@
 			)
 		)
-		(property "Footprint" "UTSVT_Connectors:Banana_Jack_1_Pin_4mm"
+		(property "Footprint" "VoltTemp:5754"
 			(at 54.61 52.07 0)
 			(effects
@@
 			)
 		)
-		(property "P/N" "105-2210-201"
+		(property "P/N" "575-4"
 			(at 54.61 52.07 90)
 			(effects
@@
 			)
 		)
-		(property "Footprint" "UTSVT_Connectors:Banana_Jack_1_Pin_4mm"
+		(property "Footprint" "VoltTemp:5754"
 			(at 140.97 71.12 0)
 			(effects
@@
 			)
 		)
-		(property "P/N" "105-2210-201"
+		(property "P/N" "575-4"
 			(at 140.97 71.12 90)
 			(effects
@@
 			)
 		)
-		(property "Footprint" "UTSVT_Connectors:Banana_Jack_1_Pin_4mm"
+		(property "Footprint" "VoltTemp:5754"
 			(at 72.39 116.84 0)
 			(effects
@@
 			)
 		)
-		(property "P/N" "105-2210-201"
+		(property "P/N" "575-4"
 			(at 72.39 116.84 0)
 			(effects
@@
 			)
 		)
-		(property "Footprint" "UTSVT_Connectors:105313-2102"
+		(property "Footprint" "UTSVT_Connectors:Molex_Nano-Fit_105309-xx02_1x02_P2.50mm_Vertical"
 			(at 185.42 69.85 0)
 			(effects
@@
 			)
 		)
-		(property "P/N" "1053131102"
+		(property "P/N" "1053091202"
 			(at 185.42 69.85 0)
 			(effects
