File: hardware/VoltTemp/TemperatureFilter.kicad_sch (KiCad schematic)
At the start: 9 parts, among them U4 TLV9062xD

Commit message: ninjafix thanks lakshay :(
Connections:
- net GNDA: now also C3.2, R35.1
- net at R1.2, R34.1: now also C25.1
- net at C3.1, R34.2, U4.5 (+): no longer C25.1
Other:
- moved on the sheet: C25, TP11
