File: hardware/VoltTemp/TemperatureFilter.kicad_sch (KiCad schematic)
At the start: 9 parts, among them U4 TLV9062xD

Commit message: Staircase (#6)
* this is the staircase board :(

* I added the 3d models for the connectors. Need to swap layers around some

* Traces finished, passes DRC, need to complete silkscreen

* changes

* Initial board done. Labels on everything, yay

* Goofy pictures and names added

* goofy things

* Review Council concerns have been dealt with :-)

* Boot switch changed to V_Boot, ShieldGND added to scrut conn, labels added to LEDs, misc routing tweaks

* i tweaked one more thing :)

* lakshay concerns dealt with and also i did the jlcpcb generation thing

* fix

* i fixed the clearance violation :-)

* STEP file generated

* board center origin

* ninjafix thanks lakshay :(

* gerbers

* bom

* bom

---------

Co-authored-by: Clark Rucker <clarkrucker@utexas.edu>
Co-authored-by: sodaplayzz <sc.seaofthieves@gmail.com>
Connections:
- net GNDA: now also C3.2, R35.1
- net at R1.2, R34.1: now also C25.1
- net at C3.1, R34.2, U4.5 (+): no longer C25.1
Other:
- moved on the sheet: C25, TP11
