File: hardware/VoltTemp/TemperatureFilter.kicad_sch (KiCad schematic)
At the start: 9 parts, among them U4 TLV9062xD

Commit message: Rev C (#21)
* rev c

* balls

* balls

* jlcpcb assembly files

* volttemp gerber stuff
Parts:
- C25: LCSC P/N (none) -> C2178293
Changed lines of the file:
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@@
-			)
-		)
-		(property "Id" ""
-			(at 149.86 48.26 0)
-			(effects
-				(font
-					(size 1.27 1.27)
-				)
-			)
-		)
-		(property "MANUFACTURER" ""
-			(at 149.86 48.26 0)
-			(effects
-				(font
-					(size 1.27 1.27)
-				)
-			)
-		)
-		(property "MAXIMUM_PACKAGE_HEIGHT" ""
-			(at 149.86 48.26 0)
-			(effects
-				(font
-					(size 1.27 1.27)
-				)
-			)
-		)
-		(property "PARTREV" ""
-			(at 149.86 48.26 0)
-			(effects
-				(font
-					(size 1.27 1.27)
-				)
-			)
-		)
-		(property "STANDARD" ""
-			(at 149.86 48.26 0)
-			(effects
-				(font
-					(size 1.27 1.27)
-				)
-			)
-		)
-		(property "Vds" ""
-			(at 149.86 48.26 0)
-			(effects
-				(font
-					(size 1.27 1.27)
-				)
 			)
 		)
@@
 			(at 149.86 48.26 90)
 			(effects
+				(font
+					(size 1.27 1.27)
+				)
+				(hide yes)
+			)
+		)
+		(property "LCSC P/N" "C2178293"
+			(at 149.86 48.26 90)
+			(effects
