File: hardware/VoltTemp/ScrutineeringConn.kicad_sch (KiCad schematic)
At the start: 3 parts, among them J1 ScrutineeringConn

Commit message: Rev C (#21)
* rev c

* balls

* balls

* jlcpcb assembly files

* volttemp gerber stuff
Connections:
- net 3&4COM renamed 1&2COM
- net 3&4COM_OUT renamed 1&2COM_OUT
Other:
- note added: "For scrutineering we're routing one thermistor output to scrut board That output will be disconnected by scrut board and a new signal injected rawTemperature4_Pre (pin 8) is an output from this board rawTemperature4 (pin 6) is an input from the scrutineering board"
- note added: "For voltage scrutineering we will pass one tap to the scrut board that tap will be disconnected for scrutineering and a new signal injected that tap will be routed back to this volttemp 1&2COM (pin 3) is an output from this board 1&2COM_OUT (pin 4) is an input from the scrutineering board"
- note removed: "For scrutineering we're routing one thermistor output to scrut board That output will be disconnected by scrut board and a new signal injected"
- note removed: "For voltage scrutineering we will pass one tap to the scrut board that tap will be disconnected for scrutineering and a new signal injected that tap will be routed back to this volttemp"
Changed lines of the file:
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@@
 	(rectangle
 		(start 91.44 43.18)
-		(end 166.37 74.93)
+		(end 166.37 83.82)
 		(stroke
 			(width 0)
@@
 	(rectangle
 		(start 16.256 43.18)
-		(end 91.44 74.93)
+		(end 91.44 83.82)
 		(stroke
 			(width 0)
@@
 		)
 	)
-	(text "For scrutineering we're routing one thermistor output to scrut board\nThat output will be disconnected by scrut board and a new signal injected"
-		(exclude_from_sim no)
-		(at 165.354 72.39 0)
+	(text "For scrutineering we're routing one thermistor output to scrut board\nThat output will be disconnected by scrut board and a new signal injected\n\nrawTemperature4_Pre (pin 8) is an output from this board\nrawTemperature4 (pin 6) is an input from the scrutineering board"
+		(exclude_from_sim no)
+		(at 165.1 73.66 0)
 		(effects
 			(font
@@
 		)
 	)
-	(text "For voltage scrutineering we will pass one tap to the scrut board\nthat tap will be disconnected for scrutineering and a new signal injected\nthat tap will be routed back to this volttemp"
-		(exclude_from_sim no)
-		(at 89.662 71.882 0)
+	(text "For voltage scrutineering we will pass one tap to the scrut board\nthat tap will be disconnected for scrutineering and a new signal injected\nthat tap will be routed back to this volttemp\n\n1&2COM (pin 3) is an output from this board\n1&2COM_OUT (pin 4) is an input from the scrutineering board"
+		(exclude_from_sim no)
+		(at 89.662 74.168 0)
 		(effects
 			(font
@@
 	(text "Only one of 8 volttemps will connect to scrut\nOther volttemps will have 0 ohm bypass"
 		(exclude_from_sim no)
-		(at 111.506 79.502 0)
+		(at 113.03 87.63 0)
 		(effects
 			(font
@@
 		)
 	)
-	(hierarchical_label "3&4COM"
+	(hierarchical_label "1&2COM"
 		(shape input)
 		(at 71.12 60.96 0)
@@
 		)
 	)
-	(hierarchical_label "3&4COM_OUT"
+	(hierarchical_label "1&2COM_OUT"
 		(shape input)
 		(at 71.12 53.34 0)
@@
 					(size 1.27 1.27)
 				)
-			)
-		)
+				(hide yes)
+			)
+		)
