File: hardware/VoltTemp/BPS-Voltage_Temp_Board.kicad_sch (KiCad schematic)
At the start: 22 parts, among them J10 53307-2471, J12 Conn_01x04, J13 Conn_01x04, J2 PeripheralCAN, J5 Logic_Analyzer

Commit message: Staircase (#6)
* this is the staircase board :(

* I added the 3d models for the connectors. Need to swap layers around some

* Traces finished, passes DRC, need to complete silkscreen

* changes

* Initial board done. Labels on everything, yay

* Goofy pictures and names added

* goofy things

* Review Council concerns have been dealt with :-)

* Boot switch changed to V_Boot, ShieldGND added to scrut conn, labels added to LEDs, misc routing tweaks

* i tweaked one more thing :)

* lakshay concerns dealt with and also i did the jlcpcb generation thing

* fix

* i fixed the clearance violation :-)

* STEP file generated

* board center origin

* ninjafix thanks lakshay :(

* gerbers

* bom

* bom

---------

Co-authored-by: Clark Rucker <clarkrucker@utexas.edu>
Co-authored-by: sodaplayzz <sc.seaofthieves@gmail.com>
Parts:
- removed J12, J13: Conn_01x04, VoltTemp:1053132104, symbol Connector_Generic:Conn_01x04
- removed MH2: MountingHole_Pad, MountingHole:MountingHole_3.2mm_M3_Pad_TopBottom, symbol Mechanical:MountingHole_Pad
- added J3, J4: Conn_01x05, VoltTemp:nanofit_01x05, symbol Connector_Generic:Conn_01x05
Connections:
- net +24V: now also J3.4 (Pin_4), J4.4 (Pin_4)
- net GND: now also J3.1 (Pin_1), J4.1 (Pin_1)
- net I-CAN_H: now also J3.3 (Pin_3), J4.3 (Pin_3)
- net I-CAN_L: now also J3.2 (Pin_2), J4.2 (Pin_2)
- net LedDin: now also J5.1 (CH0); no longer J5.5 (CH4)
- net PB14: now also J5.5 (CH4); no longer J5.3 (CH2)
- net PB15: now also J5.3 (CH2); no longer J5.1 (CH0)
- net PB3: now also J5.2 (CH1); no longer J5.6 (CH5)
- net Temperature1: now also J10.13 (ADC1_IN10); no longer J10.9 (ADC1_IN7)
- net Temperature3: now also J10.9 (ADC1_IN7); no longer J10.13 (ADC1_IN10)
- net bmsEn: now also J5.6 (CH5); no longer J5.2 (CH1)
- new net ShieldGND: J3.5 (Pin_5), J4.5 (Pin_5)
Other:
- added sheet ScrutineeringConn (ScrutineeringConn.kicad_sch)
- sheet TemperatureConn ports: added rawTemp4, rawTemp4_PRE; removed none
- sheet VoltageConn ports: added 3&4Com, 3&4Com_Out; removed none
