File: hardware/VoltTemp/VoltageSense.kicad_sch (KiCad schematic)
At the start: 34 parts, among them IC1 ISO1641BDR, SW1 BOOT, U1 EL3H7, U2 BQ7692003PW, U3 EL3H7

Commit message: rev c
Parts:
- TP1: value TP_Regout -> Regout
- TP3: value TP_bmsAlert -> bmsAlert
- TP4: value bmsGND -> SegGND
- TP6: value TP_V_Boot -> VBoot
Changed lines of the file:
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@@
 			)
 		)
-		(property "Value" "TP_V_Boot"
+		(property "Value" "VBoot"
 			(at 67.31 145.2879 0)
 			(effects
@@
 			)
 		)
-		(property "Value" "TP_Regout"
+		(property "Value" "Regout"
 			(at 110.49 116.0779 0)
 			(effects
@@
 			)
 		)
-		(property "Value" "bmsGND"
+		(property "Value" "SegGND"
 			(at 110.49 126.2379 0)
 			(effects
@@
 			)
 		)
-		(property "Value" "TP_bmsAlert"
+		(property "Value" "bmsAlert"
 			(at 125.73 116.0779 0)
 			(effects

Commit message: jlcpcb assembly files
Parts:
- R3: now not fitted
- R4: value 2kΩ -> 10kΩ; P/N CRCW06032K10FKEA -> CRCW060310K0FKEI
Other:
- note removed: "V_Boot must range from 1-3.6v for all possible cell voltages. assuming a range of 2-6v (very wide range): (1/2)2v = 1.00v (1/2)6v = 3.00v :-)"
- moved on the sheet: TP6
Changed lines of the file:
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@@
 		)
 	)
-	(text "V_Boot must range from 1-3.6v for all possible cell voltages.\nassuming a range of 2-6v (very wide range):\n(1/2)2v = 1.00v\n(1/2)6v = 3.00v  :-)\n\n"
-		(exclude_from_sim no)
-		(at 39.37 159.004 0)
-		(effects
-			(font
-				(size 0.762 0.762)
-			)
-			(justify left)
-		)
-	)
 	(text "bat and regsrc connected\n"
 		(exclude_from_sim no)
@@
 	)
 	(junction
+		(at 54.61 144.78)
+		(diameter 0)
+		(color 0 0 0 0)
+	)
+	(junction
 		(at 110.49 40.64)
 		(diameter 0)
@@
 	(wire
 		(pts
-			(xy 74.93 149.86) (xy 66.04 149.86)
-		)
-		(stroke
-			(width 0)
-			(type default)
-		)
-	)
-	(wire
-		(pts
 			(xy 191.77 111.76) (xy 189.23 111.76)
 		)
@@
 	(wire
 		(pts
-			(xy 64.77 147.32) (xy 64.77 148.59)
-		)
-		(stroke
-			(width 0)
-			(type default)
-		)
-	)
-	(wire
-		(pts
 			(xy 123.19 59.69) (xy 138.43 59.69)
 		)
@@
 	(wire
 		(pts
+			(xy 64.77 144.78) (xy 66.04 146.05)
+		)
+		(stroke
+			(width 0)
+			(type default)
+		)
+	)
+	(wire
+		(pts
 			(xy 57.15 81.28) (xy 64.77 81.28)
 		)
@@
 	(wire
 		(pts
-			(xy 110.49 31.75) (xy 110.49 35.56)
+			(xy 54.61 144.78) (xy 64.77 144.78)
 		)
 		(stroke
@@
 	(wire
 		(pts
-			(xy 168.91 116.84) (xy 168.91 119.38)
+			(xy 110.49 31.75) (xy 110.49 35.56)
 		)
 		(stroke
@@
 	(wire
 		(pts
-			(xy 201.93 35.56) (xy 204.47 35.56)
+			(xy 168.91 116.84) (xy 168.91 119.38)
 		)
 		(stroke
@@
 	(wire
 		(pts
-			(xy 66.04 149.86) (xy 64.77 148.59)
+			(xy 201.93 35.56) (xy 204.47 35.56)
 		)
 		(stroke
@@
 		)
 	)
-	(label "V_Boot"
-		(at 74.93 149.86 180)
-		(effects
-			(font
-				(size 1.27 1.27)
-			)
-			(justify right bottom)
-		)
-	)
 	(label "regout"
 		(at 118.11 120.65 180)
@@
 			)
 		)
-		(property "Value" "2kΩ"
+		(property "Value" "10kΩ"
 			(at 49.53 144.78 90)
 			(effects
@@
 			)
 		)
-		(property "P/N" "CRCW06032K10FKEA "
+		(property "P/N" "CRCW060310K0FKEI "
 			(at 49.53 144.78 0)
 			(effects
@@
 	(symbol
 		(lib_id "Connector:TestPoint")
-		(at 64.77 147.32 0)
+		(at 66.04 146.05 180)
 		(unit 1)
 		(exclude_from_sim no)
@@
 		(fields_autoplaced yes)
 		(property "Reference" "TP6"
-			(at 67.31 142.7479 0)
+			(at 68.58 148.0819 0)
 			(effects
 				(font
 					(size 1.27 1.27)
 				)
-				(justify left)
+				(justify right)
 			)
 		)
 		(property "Value" "VBoot"
-			(at 67.31 145.2879 0)
+			(at 68.58 150.6219 0)
 			(effects
 				(font
 					(size 1.27 1.27)
 				)
-				(justify left)
+				(justify right)
 			)
 		)
 		(property "Footprint" "TestPoint:TestPoint_Pad_1.0x1.0mm"
-			(at 69.85 147.32 0)
+			(at 60.96 146.05 0)
 			(effects
 				(font
@@
 		)
 		(property "Datasheet" "~"
-			(at 69.85 147.32 0)
+			(at 60.96 146.05 0)
 			(effects
 				(font
@@
 		)
 		(property "Description" "test point"
-			(at 64.77 147.32 0)
+			(at 66.04 146.05 0)
 			(effects
 				(font
@@
 		)
 		(property "Id" ""
-			(at 64.77 147.32 0)
+			(at 66.04 146.05 0)
 			(effects
 				(font
@@
 		)
 		(property "MANUFACTURER" ""
-			(at 64.77 147.32 0)
+			(at 66.04 146.05 0)
 			(effects
 				(font
@@
 		)
 		(property "MAXIMUM_PACKAGE_HEIGHT" ""
-			(at 64.77 147.32 0)
+			(at 66.04 146.05 0)
 			(effects
 				(font
@@
 		)
 		(property "PARTREV" ""
-			(at 64.77 147.32 0)
+			(at 66.04 146.05 0)
 			(effects
 				(font
@@
 		)
 		(property "STANDARD" ""
-			(at 64.77 147.32 0)
+			(at 66.04 146.05 0)
 			(effects
 				(font
@@
 		)
 		(property "Vds" ""
-			(at 64.77 147.32 0)
+			(at 66.04 146.05 0)
 			(effects
 				(font
@@
 		(in_bom yes)
 		(on_board yes)
-		(dnp no)
+		(dnp yes)
 		(property "Reference" "R3"
 			(at 52.578 151.13 90)
