File: hardware/VoltTemp/BPS-Voltage_Temp_Board.kicad_pcb (KiCad board)
At the start: 4 copper layers, 98.4 x 81.3 mm, 150 parts, among them IC1 ISO1641BDR, J1 ScrutineeringConn, J10 53307-2471, J11 Conn_01x07, J3 Conn_01x05, J4 Conn_01x05, J5 Logic_Analyzer, J8 Conn_01x06, J9 Conn_01x03, SW1 BOOT, U1 EL3H7, U12 TLV9062xD, U13 TLV9062xD, U14 TLV9062xD, U2 BQ7692003PW, U3 EL3H7, U4 TLV9062xD, U6 TLV9062xD

Commit message: jlcpcb assembly files
Parts:
- R4: value 2kΩ -> 10kΩ
Connections:
- net /VoltageConn/1&2COM renamed /ScrutineeringConn/1&2COM
- net /VoltageConn/1&2COM_Out renamed /ScrutineeringConn/1&2COM_OUT
