File: hardware/VoltTemp/FaultIndicators.kicad_sch (KiCad schematic)
At the start: 16 parts

Commit message: Rev C (#21)
* rev c

* balls

* balls

* jlcpcb assembly files

* volttemp gerber stuff
Parts:
- added R6: 0Ω, Resistor_SMD:R_0603_1608Metric_Pad0.98x0.95mm_HandSolder, symbol Device:R
Connections:
- net +3.3V: now also R6.1; no longer C10.1, C11.1, C12.1, C13.1, C14.1, C15.1, C16.1, C17.1, D2.4 (VDD), D3.4 (VDD), D4.4 (VDD), D5.4 (VDD), D6.4 (VDD), D7.4 (VDD), D8.4 (VDD), D9.4 (VDD)
- new net ws2812b_pwr: C10.1, C11.1, C12.1, C13.1, C14.1, C15.1, C16.1, C17.1, D2.4 (VDD), D3.4 (VDD), D4.4 (VDD), D5.4 (VDD), D6.4 (VDD), D7.4 (VDD), D8.4 (VDD), D9.4 (VDD), R6.2
