File: hardware/VoltTemp/TemperatureConn.kicad_sch (KiCad schematic)
At the start: 2 parts, among them J8 Conn_01x06, J9 Conn_01x03

Commit message: Rev C (#21)
* rev c

* balls

* balls

* jlcpcb assembly files

* volttemp gerber stuff
Changed lines of the file:
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@@
 		)
+	)
+	(junction
+		(at 60.96 69.85)
+		(diameter 0)
+		(color 0 0 0 0)
 	)
 	(bus_entry
@@
 	(wire
 		(pts
+			(xy 59.69 68.58) (xy 60.96 69.85)
+		)
+		(stroke
+			(width 0)
+			(type default)
+		)
+	)
+	(wire
+		(pts
 			(xy 59.69 69.85) (xy 60.96 69.85)
 		)
@@
 		)
 	)
-	(wire
-		(pts
-			(xy 59.69 69.85) (xy 59.69 71.12)
-		)
-		(stroke
-			(width 0)
-			(type default)
-		)
-	)
 	(bus
 		(pts
@@
 	)
 	(label "rawTemperature4"
-		(at 59.69 69.85 180)
+		(at 59.69 68.58 180)
 		(effects
 			(font
@@
 	(hierarchical_label "rawTemp4"
 		(shape input)
-		(at 59.69 71.12 180)
-		(effects
-			(font
+		(at 59.69 69.85 180)
+		(effects
+			(font
