File: hardware/_restore_backup_2026-08-02T12-25-25-612/PS-SegmentMonitoringBoard.kicad_sch (KiCad schematic)
At the start: 3 parts, among them J4 24V_Conn

Commit message: schematic [IN PROG]
Parts:
- removed J4: 24V_Conn, symbol Connector_Generic:Conn_01x02
- removed R22: 18k, symbol Device:R_Small
- removed R23: 10k, symbol Device:R_Small
- added J4: Seg-Mon Base Conn, symbol Connector_Generic:Conn_02x12_Counter_Clockwise
Connections:
- net +3.3V: now also J4.23 (Pin_23), J4.24 (Pin_24)
- net GND: now also J4.12 (Pin_12), J4.13 (Pin_13)
- new net +24V: J4.1 (Pin_1)
- no-connect marks 3 -> 0
Other:
- removed sheet 3.3V LDO
- removed sheet 3.3V MUX
- removed sheet USB Receptacle
- added sheet ESP32 (ESP32.kicad_sch)
- sheet 48PinMCU ports: added none; removed +3.3V, BOOT0, GND, GNDA, PA0, PA1, PA10, PA15, PA2, PA3, PA4, PA5, PA6, PA7, PA8, PA9, PB0, PB1, PB10, PB11, PB12, PB13, PB14, PB15, PB2, PB3, PB4, PB5, PB6, PB7, PB9, PC13, PC14, PC15, PG10-NRST, USB_DM, USB_DP, VDDA
- sheet Temp Sense ports: added none; removed {TEMP_THERMS}
- sheet Voltage Sense ports: added none; removed bmsAlert, {BQ_I2C}
