File: hardware/PS-SegmentMonitoringBoard.kicad_sch (KiCad schematic)
At the start: 7 parts, among them IC3 BQ79616PAPR, J2 Volt_Taps_Conn, J3 N_Conn, J4 Ring_Conn

Commit message: updated sheets and 1st review changes
Parts:
- removed C61: 10nF, symbol Device:C_Small
- removed C62: 470nF, symbol Device:C_Small
- removed J3: N_Conn, symbol Connector_Generic:Conn_01x02
- removed R28: 30, symbol Device:R_Small
- added J1: Therms_Conn, symbol Connector_Generic:Conn_01x08
- added J5: Ring_Conn, symbol Connector_Generic:Conn_01x02
- J4: value Ring_Conn -> Daisy_Chain_Conn
Connections:
- net Capacitor_Isolation_Ring/preIsolatedP: now reaches IC3.43 (COMHP)
- net Capacitor_Isolation_Ring/preIsolatedN: now reaches IC3.42 (COMHN)
- net extraCells: now reaches IC3.10 (CB12), IC3.12 (CB11), IC3.14 (CB10), IC3.16 (CB9), IC3.18 (CB8), IC3.2 (CB16), IC3.4 (CB15), IC3.6 (CB14), IC3.8 (CB13)
- net extraCells: now also IC3.11 (VC12), IC3.13 (VC11), IC3.15 (VC10), IC3.17 (VC9), IC3.19 (VC8), IC3.3 (VC16), IC3.5 (VC15), IC3.7 (VC14), IC3.9 (VC13)
- net Capacitor_Isolation_Daisy_Chain/isolatedP: now reaches J4.1 (Pin_1)
- net Capacitor_Isolation_Daisy_Chain/isolatedP: no longer IC3.40 (COMLP)
- net Capacitor_Isolation_Daisy_Chain/isolatedN: now reaches J4.2 (Pin_2)
- net Capacitor_Isolation_Daisy_Chain/isolatedN: no longer IC3.41 (COMLN)
- net GNDA renamed AVSS
- net GNDC renamed CVSS
- net GNDD renamed DVSS
- net GNDR renamed REFHM
- net GND_Bypasses/LDOIN renamed LDOIN_NPN/LDOIN
- net GND_Bypasses/NEG5V renamed NEG5V
- net GND_Bypasses/NPNB renamed LDOIN_NPN/NPNB
- removed net X_CELLS: IC3.1 (BAT), IC3.11 (VC12), IC3.13 (VC11), IC3.15 (VC10), IC3.17 (VC9), IC3.19 (VC8), IC3.3 (VC16), IC3.5 (VC15), IC3.7 (VC14), IC3.9 (VC13)
- new net Capacitor_Isolation_Daisy_Chain/preIsolatedN: IC3.41 (COMLN)
- new net Capacitor_Isolation_Daisy_Chain/preIsolatedP: IC3.40 (COMLP)
- new net Capacitor_Isolation_Ring/isolatedN: J5.2 (Pin_2)
- new net Capacitor_Isolation_Ring/isolatedP: J5.1 (Pin_1)
- new net TEMP_0: J1.1 (Pin_1)
- new net TEMP_1: J1.2 (Pin_2)
- new net TEMP_2: J1.3 (Pin_3)
- new net TEMP_3: J1.4 (Pin_4)
- new net TEMP_4: J1.5 (Pin_5)
- new net TEMP_5: J1.6 (Pin_6)
- new net TEMP_6: J1.7 (Pin_7)
- new net TEMP_7: J1.8 (Pin_8)
- new net preBAT: IC3.1 (BAT)
Other:
- added sheet Capacitor_Isolation_Daisy_Chain (Capacitor_Isolation.kicad_sch)
- added sheet Capacitor_Isolation_Ring (Capacitor_Isolation.kicad_sch)
- added sheet Cell_Balancing (Cell_Balancing.kicad_sch)
- added sheet Extra_Cells (Extra_Cells.kicad_sch)
- added sheet LDOIN_NPN (LDOIN_NPN.kicad_sch)
- sheet GND_Bypasses ports: added AVSS, CVSS, DVSS, REFHM; removed BAT, GNDA, GNDC, GNDD, GNDR, LDOIN, NPNB
- sheet Thermistors ports: added AVSS, {TEMPS}; removed CVDD, GNDA
- sheet Volt_Taps ports: added AVSS; removed GNDA, {CELL_BALANCING}
- note added: "Major Todo's: - redo resistor math for 240mA -> DONE - figure out NFAULT -> im p sure we dont need - double check whether I need NTC filters or not -> DONE - cap isolation with choke shi -> DONE"
- moved on the sheet: J2, J4

Commit message: updated sheets, footprint, and calcs; 2nd review changes
Parts:
- removed IC3: BQ79616PAPR, QFP50P1200X1200X120-65N, symbol custom_symbols:BQ79616PAPR
- added C1, C2: 1uF, Capacitor_SMD:C_0201_0603Metric_Pad0.64x0.40mm_HandSolder, symbol Device:C_Small
- added C3: 22nF, Capacitor_SMD:C_0201_0603Metric_Pad0.64x0.40mm_HandSolder, symbol Device:C_Small
- added C4: 4.7uF, Capacitor_SMD:C_0805_2012Metric_Pad1.18x1.45mm_HandSolder, symbol Device:C_Small
- added C5: 100nF, Capacitor_SMD:C_0201_0603Metric_Pad0.64x0.40mm_HandSolder, symbol Device:C_Small
- added C6: 2.2uF, Capacitor_SMD:C_0805_2012Metric_Pad1.18x1.45mm_HandSolder, symbol Device:C_Small
- added C7: 0.1uF, Capacitor_SMD:C_0603_1608Metric_Pad1.08x0.95mm_HandSolder, symbol Device:C_Small
- added IC1: BQ79616PAPR, QFP50P1200X1200X120-65N, symbol Custom-KiCAD-Lib:BQ79616PAPR
- J1: renamed from J2; value Volt_Taps_Conn -> voltTapsConn; footprint (none) -> Custom-Footprints:1054301108
- J2: renamed from J5; value Ring_Conn -> highSideConn; footprint (none) -> Custom-Footprints:1054301102
- J3: renamed from J4; value Daisy_Chain_Conn -> lowSideConn; footprint (none) -> Custom-Footprints:1054301102
- J4: renamed from J1; value Therms_Conn -> thermsConn; footprint (none) -> Custom-Footprints:1054301108
Connections:
- net AVSS: now also C1.2, C2.2, C3.2, C4.2, C5.2, C6.2, C7.2, IC1.36 (REFHM), IC1.39 (AVSS), IC1.46 (CVSS), IC1.50 (DVSS), IC1.65 (PAD)
- net CB0: now also IC1.34 (CB0)
- net CB1: now also IC1.32 (CB1)
- net CB2: now also IC1.30 (CB2)
- net CB3: now also IC1.28 (CB3)
- net CB4: now also IC1.26 (CB4)
- net CB5: now also IC1.24 (CB5)
- net CB6: now also IC1.22 (CB6)
- net CB7: now also IC1.20 (CB7)
- net CVDD: now also C4.1, IC1.45 (CVDD), IC1.52 (RX)
- net LDOIN_NPN/LDOIN: now also IC1.47 (LDOIN)
- net LDOIN_NPN/NPNB: now also IC1.48 (NPNB)
- net NTC0: now also IC1.61 (GPIO1)
- net NTC1: now also IC1.60 (GPIO2)
- net NTC2: now also IC1.59 (GPIO3)
- net NTC3: now also IC1.58 (GPIO4)
- net NTC4: now also IC1.57 (GPIO5)
- net NTC5: now also IC1.56 (GPIO6)
- net NTC6: now also IC1.55 (GPIO7)
- net NTC7: now also IC1.54 (GPIO8)
- net TSREF: now also IC1.51 (TSREF)
- net VC0: now also IC1.35 (VC0)
- net VC1: now also IC1.33 (VC1)
- net VC2: now also IC1.31 (VC2)
- net VC3: now also IC1.29 (VC3)
- net VC4: now also IC1.27 (VC4)
- net VC5: now also IC1.25 (VC5)
- net VC6: now also IC1.23 (VC6)
- net VC7: now also IC1.21 (VC7)
- net extraCells: now also IC1.1 (BAT), IC1.10 (CB12), IC1.11 (VC12), IC1.12 (CB11), IC1.13 (VC11), IC1.14 (CB10), IC1.15 (VC10), IC1.16 (CB9), IC1.17 (VC9), IC1.18 (CB8), IC1.19 (VC8), IC1.2 (CB16), IC1.3 (VC16), IC1.4 (CB15), IC1.5 (VC15), IC1.6 (CB14), IC1.7 (VC14), IC1.8 (CB13), IC1.9 (VC13)
- net lowSideIsolation/isolatedN renamed lowSideIsolation/isolatedCOMLN
- net lowSideIsolation/isolatedP renamed lowSideIsolation/isolatedCOMLP
- net highSideIsolation/isolatedN renamed highSideIsolation/isolatedCOMHN
- net highSideIsolation/isolatedP renamed highSideIsolation/isolatedCOMHP
- new net: C3.1, C5.1
- new net: C2.1, IC1.38 (AVDD)
- new net: C1.1, IC1.37 (REFHP)
- new net: C7.1, IC1.44 (NEG5V)
- new net: C6.1, IC1.49 (DVDD)
- new net highSideIsolation/COMHN: IC1.42 (COMHN)
- new net highSideIsolation/COMHP: IC1.43 (COMHP)
- new net lowSideIsolation/COMLN: IC1.41 (COMLN)
- new net lowSideIsolation/COMLP: IC1.40 (COMLP)
Other:
- sheet Capacitor_Isolation_Daisy_Chain renamed lowSideIsolation
- sheet Capacitor_Isolation_Ring renamed highSideIsolation
- removed sheet Extra_Cells
- removed sheet GND_Bypasses
- sheet LDOIN_NPN ports: added V7; removed BAT
- sheet Thermistors ports: added {NTCS}; removed NTCS
- sheet Volt_Taps ports: added extraCells; removed none
- sheet highSideIsolation: file Capacitor_Isolation.kicad_sch -> highSideIsolation.kicad_sch
- sheet highSideIsolation ports: added COMHN, COMHP, isolatedCOMHN, isolatedCOMHP; removed isolatedN, isolatedP, preIsolatedN, preIsolatedP
- sheet lowSideIsolation: file Capacitor_Isolation.kicad_sch -> lowSideIsolation.kicad_sch
- sheet lowSideIsolation ports: added COMLN, COMLP, isolatedCOMLN, isolatedCOMLP; removed isolatedN, isolatedP, preIsolatedN, preIsolatedP
- moved on the sheet: J1, J4
