File: hardware/5V_Buck.kicad_sch (KiCad schematic)
At the start: 12 parts, among them U1 LMR51635XDDCR

Commit message: schem except BQ
Parts:
- C2: footprint Resistor_SMD:R_0201_0603Metric_Pad0.64x0.40mm_HandSolder -> Capacitor_SMD:C_0603_1608Metric
- L1: value 5.6u -> 10u; footprint Inductor_SMD:L_TDK_SLF6025 -> Inductor_SMD:L_TDK_VLP8040; LCSC P/N C2997651 -> C354639; P/N PNLS6045-5R6M 5.6UH -> CKCS8040-10uH/M
- R1: value 31.6k -> 53.6k; LCSC P/N C25967 -> C23074; P/N 0603WAF3162T5E -> 0603WAF5362T5E
- U1: footprint breh:DDC0006A-MFG -> utsvt_ics:DDC0006A-MFG
Connections:
- net V_out_3V3 renamed V_out_5V
Other:
- note added: "24V-5V Buck Converter"
- note added: "5V Vout"
- note removed: "24V-3.3V Buck Converter"
- note removed: "3.3V Vout"
