File: hardware/5V_MUX.kicad_sch (KiCad schematic)
At the start: 6 parts, among them U6 TPS2117DRLR

Commit message: schem except BQ
Parts:
- renumbered C29 to C27, C30 to C28, C31 to C29, C32 to C30, U6 to U3
Other:
- moved on the sheet: C27, C28, C29, C30, R21, U3
