File: hardware/USB.kicad_sch (KiCad schematic)
At the start: 5 parts, among them J7 USB_C_Receptacle_USB2.0_16P

Commit message: schem except BQ
Connections:
- net USB_D+: now also J7.A7 (D-), J7.B7 (D-); no longer J7.A6 (D+), J7.B6 (D+)
- net USB_D-: now also J7.A6 (D+), J7.B6 (D+); no longer J7.A7 (D-), J7.B7 (D-)
Changed lines of the file:
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@@
 	(paper "A4")
 	(junction
+		(at 160.02 46.99)
+		(diameter 0)
+		(color 0 0 0 0)
+	)
+	(junction
+		(at 154.94 54.61)
+		(diameter 0)
+		(color 0 0 0 0)
+	)
+	(junction
+		(at 137.16 64.77)
+		(diameter 0)
+		(color 0 0 0 0)
+	)
+	(junction
+		(at 120.65 86.36)
+		(diameter 0)
+		(color 0 0 0 0)
+	)
+	(junction
 		(at 137.16 62.23)
-		(diameter 0)
-		(color 0 0 0 0)
-	)
-	(junction
-		(at 160.02 46.99)
-		(diameter 0)
-		(color 0 0 0 0)
-	)
-	(junction
-		(at 137.16 64.77)
-		(diameter 0)
-		(color 0 0 0 0)
-	)
-	(junction
-		(at 120.65 86.36)
-		(diameter 0)
-		(color 0 0 0 0)
-	)
-	(junction
-		(at 152.4 54.61)
 		(diameter 0)
 		(color 0 0 0 0)
@@
 		(at 135.89 77.47)
 	)
-	(bus_entry
-		(at 147.32 62.23)
-		(size 2.54 2.54)
-		(stroke
-			(width 0)
-			(type default)
-		)
-	)
-	(bus_entry
-		(at 147.32 64.77)
-		(size 2.54 2.54)
-		(stroke
-			(width 0)
-			(type default)
-		)
-	)
 	(wire
 		(pts
@@
 	(wire
 		(pts
-			(xy 152.4 54.61) (xy 152.4 52.07)
+			(xy 154.94 54.61) (xy 154.94 52.07)
 		)
 		(stroke
@@
 		)
 	)
-	(bus
-		(pts
-			(xy 149.86 64.77) (xy 149.86 69.85)
-		)
-		(stroke
-			(width 0)
-			(type default)
-		)
-	)
 	(wire
 		(pts
@@
 		)
 	)
-	(bus
-		(pts
-			(xy 149.86 69.85) (xy 158.75 69.85)
-		)
-		(stroke
-			(width 0)
-			(type default)
-		)
-	)
 	(wire
 		(pts
@@
 	(wire
 		(pts
-			(xy 152.4 54.61) (xy 152.4 57.15)
-		)
-		(stroke
-			(width 0)
-			(type default)
-		)
-	)
-	(wire
-		(pts
-			(xy 152.4 52.07) (xy 147.32 52.07)
+			(xy 154.94 54.61) (xy 154.94 55.88)
+		)
+		(stroke
+			(width 0)
+			(type default)
+		)
+	)
+	(wire
+		(pts
+			(xy 154.94 52.07) (xy 147.32 52.07)
 		)
 		(stroke
@@
 	(wire
 		(pts
-			(xy 137.16 62.23) (xy 147.32 62.23)
+			(xy 147.32 54.61) (xy 154.94 54.61)
+		)
+		(stroke
+			(width 0)
+			(type default)
+		)
+	)
+	(wire
+		(pts
+			(xy 137.16 62.23) (xy 140.97 62.23)
 		)
 		(stroke
@@
 	(wire
 		(pts
-			(xy 137.16 64.77) (xy 147.32 64.77)
+			(xy 137.16 64.77) (xy 140.97 64.77)
 		)
 		(stroke
@@
 			(width 0)
 			(type default)
-		)
-	)
-	(wire
-		(pts
-			(xy 147.32 54.61) (xy 152.4 54.61)
-		)
-		(stroke
-			(width 0)
-			(type default)
-		)
-	)
-	(label "USB_D+"
-		(at 147.32 64.77 180)
-		(effects
-			(font
-				(size 1.27 1.27)
-			)
-			(justify right bottom)
 		)
 	)
@@
 		)
 	)
-	(label "USB_D-"
-		(at 147.32 62.23 180)
-		(effects
-			(font
-				(size 1.27 1.27)
-			)
-			(justify right bottom)
-		)
-	)
 	(hierarchical_label "GND"
 		(shape bidirectional)
-		(at 152.4 57.15 270)
+		(at 154.94 55.88 270)
 		(effects
 			(font
@@
 		)
 	)
-	(hierarchical_label "{USB}"
-		(shape output)
-		(at 158.75 69.85 0)
+	(hierarchical_label "USB_D-"
+		(shape bidirectional)
+		(at 140.97 64.77 0)
 		(effects
 			(font
@@
 		)
 	)
+	(hierarchical_label "USB_D+"
+		(shape bidirectional)
+		(at 140.97 62.23 0)
+		(effects
+			(font
+				(size 1.27 1.27)
+			)
+			(justify left)
+		)
+	)
