File: hardware/Capacitor_Isolation.kicad_sch (KiCad schematic)
At the start: 7 parts

Commit message: updated sheets, footprint, and calcs; 2nd review changes
Parts:
- renumbered C13 to C1, C14 to C2, C6 to C3, R4 to R1, R5 to R2, R6 to R3
Connections:
- no-connect marks 0 -> 1
Changed lines of the file:
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@@
 		(color 0 0 0 0)
+	)
+	(no_connect
+		(at 171.45 49.53)
 	)
 	(wire
@@
 		(in_pos_files yes)
 		(dnp no)
-		(property "Reference" "C6"
+		(property "Reference" "C3"
 			(at 157.734 48.514 90)
 			(show_name no)
@@
 			(project "PS-SegmentMonitoringBoard"
 				(path "/f5c3f134-fd91-4d3b-aae6-719b554b2d69/b9160b78-ad79-4299-ac76-fc3d5563367b"
-					(reference "C6")
+					(reference "C3")
 					(unit 1)
 				)
 				(path "/f5c3f134-fd91-4d3b-aae6-719b554b2d69/d92b970b-7f5c-4231-93c3-49a40e55038f"
-					(reference "C16")
+					(reference "C18")
 					(unit 1)
 				)
@@
 		(in_pos_files yes)
 		(dnp no)
-		(property "Reference" "#PWR01"
+		(property "Reference" "#PWR017"
 			(at 152.4 55.88 0)
 			(hide yes)
@@
 			(project "PS-SegmentMonitoringBoard"
 				(path "/f5c3f134-fd91-4d3b-aae6-719b554b2d69/b9160b78-ad79-4299-ac76-fc3d5563367b"
-					(reference "#PWR01")
+					(reference "#PWR017")
 					(unit 1)
 				)
 				(path "/f5c3f134-fd91-4d3b-aae6-719b554b2d69/d92b970b-7f5c-4231-93c3-49a40e55038f"
-					(reference "#PWR02")
+					(reference "#PWR018")
 					(unit 1)
 				)
@@
 		(dnp no)
 		(fields_autoplaced yes)
-		(property "Reference" "C14"
+		(property "Reference" "C2"
 			(at 130.81 60.9662 0)
 			(show_name no)
@@
 			(project "PS-SegmentMonitoringBoard"
 				(path "/f5c3f134-fd91-4d3b-aae6-719b554b2d69/b9160b78-ad79-4299-ac76-fc3d5563367b"
-					(reference "C14")
+					(reference "C2")
 					(unit 1)
 				)
 				(path "/f5c3f134-fd91-4d3b-aae6-719b554b2d69/d92b970b-7f5c-4231-93c3-49a40e55038f"
-					(reference "C4")
+					(reference "C17")
 					(unit 1)
 				)
@@
 		(dnp no)
 		(fields_autoplaced yes)
-		(property "Reference" "C13"
+		(property "Reference" "C1"
 			(at 130.81 43.1862 0)
 			(show_name no)
@@
 			(project "PS-SegmentMonitoringBoard"
 				(path "/f5c3f134-fd91-4d3b-aae6-719b554b2d69/b9160b78-ad79-4299-ac76-fc3d5563367b"
-					(reference "C13")
+					(reference "C1")
 					(unit 1)
 				)
 				(path "/f5c3f134-fd91-4d3b-aae6-719b554b2d69/d92b970b-7f5c-4231-93c3-49a40e55038f"
-					(reference "C3")
+					(reference "C16")
 					(unit 1)
 				)
@@
 		(dnp no)
 		(fields_autoplaced yes)
-		(property "Reference" "R5"
+		(property "Reference" "R2"
 			(at 144.78 35.56 90)
 			(show_name no)
@@
 			(project "PS-SegmentMonitoringBoard"
 				(path "/f5c3f134-fd91-4d3b-aae6-719b554b2d69/b9160b78-ad79-4299-ac76-fc3d5563367b"
-					(reference "R5")
+					(reference "R2")
 					(unit 1)
 				)
 				(path "/f5c3f134-fd91-4d3b-aae6-719b554b2d69/d92b970b-7f5c-4231-93c3-49a40e55038f"
-					(reference "R2")
+					(reference "R16")
 					(unit 1)
 				)
@@
 		(dnp no)
 		(fields_autoplaced yes)
-		(property "Reference" "R4"
+		(property "Reference" "R1"
 			(at 116.84 48.2599 0)
 			(show_name no)
@@
 			(project "PS-SegmentMonitoringBoard"
 				(path "/f5c3f134-fd91-4d3b-aae6-719b554b2d69/b9160b78-ad79-4299-ac76-fc3d5563367b"
-					(reference "R4")
+					(reference "R1")
 					(unit 1)
 				)
 				(path "/f5c3f134-fd91-4d3b-aae6-719b554b2d69/d92b970b-7f5c-4231-93c3-49a40e55038f"
-					(reference "R1")
+					(reference "R15")
 					(unit 1)
 				)
@@
 		(dnp no)
 		(fields_autoplaced yes)
-		(property "Reference" "R6"
+		(property "Reference" "R3"
 			(at 144.78 53.34 90)
 			(show_name no)
@@
 			(project "PS-SegmentMonitoringBoard"
 				(path "/f5c3f134-fd91-4d3b-aae6-719b554b2d69/b9160b78-ad79-4299-ac76-fc3d5563367b"
-					(reference "R6")
-					(unit 1)
-				)
-				(path "/f5c3f134-fd91-4d3b-aae6-719b554b2d69/d92b970b-7f5c-4231-93c3-49a40e55038f"
 					(reference "R3")
 					(unit 1)
 				)
+				(path "/f5c3f134-fd91-4d3b-aae6-719b554b2d69/d92b970b-7f5c-4231-93c3-49a40e55038f"
+					(reference "R17")
+					(unit 1)
+				)
