File: hardware/LDOIN_NPN.kicad_sch (KiCad schematic)
At the start: 5 parts, among them Q1 NPN

Commit message: updated sheets, footprint, and calcs; 2nd review changes
Parts:
- C22: renamed from C132; footprint (none) -> Capacitor_SMD:C_0603_1608Metric_Pad1.08x0.95mm_HandSolder
- C23: renamed from C131; footprint (none) -> Capacitor_SMD:C_0603_1608Metric_Pad1.08x0.95mm_HandSolder
- Q1: footprint (none) -> Custom-Footprints:ZXTN4004KTC
- R12: renamed from R98; footprint (none) -> Resistor_SMD:R_0805_2012Metric_Pad1.20x1.40mm_HandSolder
- R13: renamed from R97; footprint (none) -> Resistor_SMD:R_0805_2012Metric_Pad1.20x1.40mm_HandSolder
Connections:
- net BAT renamed V7
Changed lines of the file:
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@@
 		)
 	)
-	(hierarchical_label "BAT"
+	(hierarchical_label "V7"
 		(shape input)
 		(at 101.6 105.41 180)
@@
 		(dnp no)
 		(fields_autoplaced yes)
-		(property "Reference" "R98"
+		(property "Reference" "R12"
 			(at 109.22 100.33 90)
 			(show_name no)
@@
 			)
 		)
-		(property "Footprint" ""
+		(property "Footprint" "Resistor_SMD:R_0805_2012Metric_Pad1.20x1.40mm_HandSolder"
 			(at 109.22 105.41 0)
 			(hide yes)
@@
 			(project "PS-SegmentMonitoringBoard"
 				(path "/f5c3f134-fd91-4d3b-aae6-719b554b2d69/0f5bcfdc-20b6-4bf4-b7a4-a429fefce66c"
-					(reference "R98")
+					(reference "R12")
 					(unit 1)
 				)
@@
 		(in_pos_files yes)
 		(dnp no)
-		(property "Reference" "C132"
+		(property "Reference" "C22"
 			(at 129.794 109.982 0)
 			(show_name no)
@@
 			)
 		)
-		(property "Footprint" ""
+		(property "Footprint" "Capacitor_SMD:C_0603_1608Metric_Pad1.08x0.95mm_HandSolder"
 			(at 127 111.76 0)
 			(hide yes)
@@
 			(project "PS-SegmentMonitoringBoard"
 				(path "/f5c3f134-fd91-4d3b-aae6-719b554b2d69/0f5bcfdc-20b6-4bf4-b7a4-a429fefce66c"
-					(reference "C132")
+					(reference "C22")
 					(unit 1)
 				)
@@
 		(dnp no)
 		(fields_autoplaced yes)
-		(property "Reference" "R97"
+		(property "Reference" "R13"
 			(at 119.38 100.33 90)
 			(show_name no)
@@
 			)
 		)
-		(property "Footprint" ""
+		(property "Footprint" "Resistor_SMD:R_0805_2012Metric_Pad1.20x1.40mm_HandSolder"
 			(at 119.38 105.41 0)
 			(hide yes)
@@
 			(project "PS-SegmentMonitoringBoard"
 				(path "/f5c3f134-fd91-4d3b-aae6-719b554b2d69/0f5bcfdc-20b6-4bf4-b7a4-a429fefce66c"
-					(reference "R97")
+					(reference "R13")
 					(unit 1)
 				)
@@
 			)
 		)
-		(property "Footprint" ""
+		(property "Footprint" "Custom-Footprints:ZXTN4004KTC"
 			(at 142.24 166.37 0)
 			(hide yes)
@@
 		(in_pos_files yes)
 		(dnp no)
-		(property "Reference" "C131"
+		(property "Reference" "C23"
 			(at 161.544 109.982 0)
 			(show_name no)
@@
 			)
 		)
-		(property "Footprint" ""
+		(property "Footprint" "Capacitor_SMD:C_0603_1608Metric_Pad1.08x0.95mm_HandSolder"
 			(at 158.75 111.76 0)
 			(hide yes)
@@
 			(project "PS-SegmentMonitoringBoard"
 				(path "/f5c3f134-fd91-4d3b-aae6-719b554b2d69/0f5bcfdc-20b6-4bf4-b7a4-a429fefce66c"
-					(reference "C131")
+					(reference "C23")
 					(unit 1)
 				)
